Commit message: updated URDF files for RGB-D camera

File: my_robot/urdf/my_robot.xacro (robot description, xacro)
@@ -166,4 +166,11 @@
     <material>Gazebo/Red</material>
   </gazebo>
+  <!-- RGB-D Camera -->
+  <link name="camera_link_optical"/>
+  <joint name="camera_optical_joint" type="fixed">
+    <origin xyz="0 0 0" rpy="-1.5707 0 -1.5707"/>
+    <parent link="camera"/>
+    <child link="camera_link_optical"/>
+  </joint>
   <!-- Lidar -->
   <link name="hokuyo">
